Commit message: Edit visualization

File: agv_description/urdf/agv.urdf (robot description, URDF)
Before this commit: robot rover_description, 1 links, 0 joints
Links:
- added link laser_back; visual box size=0.155 0.155 0.19
- added link laser_front; visual box size=0.155 0.155 0.19
- link base_link: geometry visual mesh filename=package://agv_description/meshes/agv1.stl
Joints:
- added joint base_link_to_laser_1: type fixed, parent base_link, child laser_front, origin xyz=0.3175 0 0.315 rpy=0 0 0
- added joint base_link_to_laser_2: type fixed, parent base_link, child laser_back, origin xyz=-0.3175 0 0.315 rpy=0 0 3.14
